File: plain60-flex-edition.kicad_sch (KiCad schematic)
At the start: 173 parts, among them J1 HRO-TYPE-C-31-M-12, J2 ISP, J3 ai03_ud, K1 KEYSW, K10 KEYSW, K11 KEYSW, K12 KEYSW, K13 KEYSW, K14 KEYSW, K15 KEYSW, K15-1 KEYSW, K16 KEYSW, K17 KEYSW, K18 KEYSW, K19 KEYSW, K2 KEYSW, K20 KEYSW, K21 KEYSW, K22 KEYSW, K23 KEYSW, K24 KEYSW, K25 KEYSW, K26 KEYSW, K27 KEYSW, K28 KEYSW, K29 KEYSW, K3 KEYSW, K31 KEYSW, K31-1 KEYSW, K32 KEYSW, K33 KEYSW, K34 KEYSW, K35 KEYSW, K36 KEYSW, K37 KEYSW, K38 KEYSW, K39 KEYSW, K4 KEYSW, K40 KEYSW, K41 KEYSW, K42 KEYSW, K43 KEYSW, K44 KEYSW, K44-1 KEYSW, K46 KEYSW, K46-1 KEYSW, K47 KEYSW, K48 KEYSW, K49 KEYSW, K5 KEYSW, K50 KEYSW, K51 KEYSW, K52 KEYSW, K53 KEYSW, K54 KEYSW, K55 KEYSW, K56 KEYSW, K57 KEYSW, K58 KEYSW, K58-1 KEYSW, K59 KEYSW, K6 KEYSW, K61 KEYSW, K61-1 KEYSW, K62 KEYSW, K62-1 KEYSW, K63 KEYSW, K63-1 KEYSW, K67 KEYSW, K67-1 KEYSW, K7 KEYSW, K71 KEYSW, K72 KEYSW, K72-1 KEYSW, K73 KEYSW, K73-1 KEYSW, K74 KEYSW, K74-1 KEYSW, K8 KEYSW, K9 KEYSW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

Commit message: Rotate enter stabilizer, not shift
Parts:
- K44: footprint Keeb_switches:CHERRY_PCB_225H -> Keeb_switches:CHERRY_PCB_225H_F
- K58: footprint Keeb_switches:CHERRY_PCB_275H_F -> Keeb_switches:CHERRY_PCB_275H
Changed lines of the file:
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@@
   (junction (at 316.23 146.05))
   (junction (at 331.47 140.97))
+  (no_connect (at 229.87 38.1))
   (no_connect (at 229.87 31.75))
   (no_connect (at 229.87 44.45))
-  (no_connect (at 44.45 74.93))
-  (no_connect (at 229.87 38.1))
+  (no_connect (at 44.45 90.17))
+  (no_connect (at 229.87 25.4))
   (no_connect (at 132.08 35.56))
+  (no_connect (at 255.27 25.4))
   (no_connect (at 229.87 57.15))
-  (no_connect (at 255.27 31.75))
+  (no_connect (at 44.45 74.93))
   (no_connect (at 255.27 38.1))
   (no_connect (at 229.87 50.8))
-  (no_connect (at 44.45 90.17))
-  (no_connect (at 229.87 25.4))
-  (no_connect (at 255.27 25.4))
+  (no_connect (at 255.27 31.75))
   (wire (pts (xy 21.59 156.21) (xy 29.21 156.21)))
   (wire (pts (xy 21.59 171.45) (xy 29.21 171.45)))
@@
       (effects (font (size 1.524 1.524)) hide)
     )
-    (property "Footprint" "Keeb_switches:CHERRY_PCB_275H_F" (id 2) (at 283.21 201.93 0)
+    (property "Footprint" "Keeb_switches:CHERRY_PCB_275H" (id 2) (at 283.21 201.93 0)
       (effects (font (size 1.524 1.524)) hide)
     )
@@
       (effects (font (size 1.524 1.524)) hide)
     )
-    (property "Footprint" "Keeb_switches:CHERRY_PCB_225H" (id 2) (at 303.53 181.61 0)
+    (property "Footprint" "Keeb_switches:CHERRY_PCB_225H_F" (id 2) (at 303.53 181.61 0)
       (effects (font (size 1.524 1.524)) hide)
     )
